File: dsp1_stm32/dsp1_stm32.kicad_pcb (KiCad board)
At the start: 2 copper layers, 112 parts, among them J1 Conn_01x04_Pin, J10 Conn_01x04_Socket, J11 Jack-DC, J12 AudioJack3, J13 Conn_01x04_Socket, J14 Conn_01x02_Pin, J15 Conn_01x02_Pin, J16 Conn_01x02_Pin, J17 Conn_01x02_Pin, J18 Conn_01x03_Pin, J2 Conn_01x04_Pin, J3 Conn_01x04_Pin, J4 USB_C_Receptacle_USB2.0_14P, J5 AudioJack3, J6 AudioJack3, J7 AudioJack3, J8 Conn_01x04_Socket, J9 Conn_01x04_Socket, SW1 SW_Push, SW10 SW_Push, SW2 SW_SPDT, SW3 SW_SPDT, SW4 SW_SPDT, SW5 SW_SPDT, SW6 SW_SPDT, SW7 SW_Push, SW8 SW_Push, SW9 SW_Push, U1 STM32H757IITx, U10 USBLC6-2SC6, U11 USBLC6-2SC6, U12 USBLC6-2SC6, U13 TLV62568DBV, U14 TLV62568DBV, U2 USBLC6-2SC6, U3 USBLC6-2SC6, U4 USBLC6-2SC6, U5 USBLC6-2SC6, U6 USBLC6-2SC6, U7 USBLC6-2SC6, U8 WE-TVS-824015043, U9 USBLC6-2SC6, Y1 25MHz

Commit message: PCB dsp v1 done
Parts:
- removed C12, C14, C15, C17: 4.7u, Capacitor_SMD:C_0603_1608Metric
- removed C31, C34: 100n, Capacitor_SMD:C_0603_1608Metric
- removed the J4 at (245.5, 99.1)
- removed the R6 at (232.8, 92.0)
- removed the R7 at (236.7, 92.0)
- removed the U5 at (236.0, 100.0)
- removed the U7 at (149.9, 136.6)
- removed the U8 at (164.1, 136.6)
- added J12: Conn_01x03_Pin, Connector_PinHeader_2.54mm:PinHeader_1x03_P2.54mm_Vertical, F.Cu at (209.5, 64.0)
- added R16: 5.1k, Resistor_SMD:R_0603_1608Metric, F.Cu at (218.9, 112.6)
- added R17: 5.1k, Resistor_SMD:R_0603_1608Metric, F.Cu at (218.9, 104.0)
- added U10: USBLC6-2SC6, Package_TO_SOT_SMD:SOT-23-6, F.Cu at (107.1, 129.0)
- added U11: WE-TVS-824015043, Package_TO_SOT_SMD:SOT-23-6, F.Cu at (119.0, 135.0)
- added U14: USBLC6-2SC6, Package_TO_SOT_SMD:SOT-23-6, F.Cu at (216.8, 107.9)
- added U15: WE-TVS-824015043, Package_TO_SOT_SMD:SOT-23-6, F.Cu at (201.9, 69.5)
- J11: value Jack-DC -> Conn_01x03_Pin; footprint Connector_BarrelJack:BarrelJack_SwitchcraftConxall_RAPC10U_Horizontal -> Connector_PinHeader_2.54mm:PinHeader_1x03_P2.54mm_Vertical
- J13: value Conn_01x04_Socket -> Conn_01x03_Pin; footprint Connector_PinSocket_2.54mm:PinSocket_1x04_P2.54mm_Vertical -> Connector_PinHeader_2.54mm:PinHeader_1x03_P2.54mm_Vertical
- J14: value Conn_01x02_Pin -> Conn_01x03_Pin; footprint Connector_PinHeader_2.54mm:PinHeader_1x02_P2.54mm_Vertical -> Connector_PinHeader_2.54mm:PinHeader_1x03_P2.54mm_Vertical
- J15: value Conn_01x02_Pin -> Conn_01x04_Pin; footprint Connector_PinHeader_2.54mm:PinHeader_1x02_P2.54mm_Vertical -> Connector_PinHeader_2.54mm:PinHeader_1x04_P2.54mm_Vertical
- J16: value Conn_01x02_Pin -> USB_C_Receptacle_USB2.0_14P; footprint Connector_PinHeader_2.54mm:PinHeader_1x02_P2.54mm_Vertical -> Connector_USB:USB_C_Receptacle_GCT_USB4105-xx-A_16P_TopMnt_Horizontal
- J17: value Conn_01x02_Pin -> Jack-DC; footprint Connector_PinHeader_2.54mm:PinHeader_1x02_P2.54mm_Vertical -> Connector_BarrelJack:BarrelJack_Horizontal
- SW1: footprint Button_Switch_SMD:SW_Push_1P1T_NO_CK_KMR2 -> Button_Switch_SMD:SW_SPST_PTS647_Sx38
- SW10: renamed from SW6; footprint Button_Switch_SMD:Nidec_Copal_CAS-120A -> Button_Switch_SMD:SW_SPDT_PCM12
- SW2: footprint Button_Switch_SMD:Nidec_Copal_CAS-120A -> Button_Switch_SMD:SW_SPDT_PCM12
- SW3: renamed from SW7; footprint Button_Switch_SMD:SW_Push_1P1T_NO_CK_KMR2 -> Button_Switch_SMD:SW_SPST_PTS647_Sx38
- SW4: renamed from SW8; footprint Button_Switch_SMD:SW_Push_1P1T_NO_CK_KMR2 -> Button_Switch_SMD:SW_SPST_PTS647_Sx38
- SW5: renamed from SW9; footprint Button_Switch_SMD:SW_Push_1P1T_NO_CK_KMR2 -> Button_Switch_SMD:SW_SPST_PTS647_Sx38
- SW6: renamed from SW10; footprint Button_Switch_SMD:SW_Push_1P1T_NO_CK_KMR2 -> Button_Switch_SMD:SW_SPST_PTS647_Sx38
- SW7: renamed from SW3; footprint Button_Switch_SMD:Nidec_Copal_CAS-120A -> Button_Switch_SMD:SW_SPDT_PCM12
- SW8: renamed from SW4; footprint Button_Switch_SMD:Nidec_Copal_CAS-120A -> Button_Switch_SMD:SW_SPDT_PCM12
- SW9: renamed from SW5; footprint Button_Switch_SMD:Nidec_Copal_CAS-120A -> Button_Switch_SMD:SW_SPDT_PCM12
- moved C35 188.3 mm to (224.5, 63.7), turned to -90 degrees
- moved C29 181.7 mm to (212.5, 77.2), turned to 90 degrees
- moved C24 172.9 mm to (189.7, 99.0)
- moved C25 167.0 mm to (189.8, 102.5)
- moved C32 160.8 mm to (189.8, 95.5)
- moved C21 135.0 mm to (151.5, 93.2), turned to -90 degrees
- moved C23 132.7 mm to (151.5, 104.3), turned to -90 degrees
- moved C20 131.1 mm to (144.3, 113.5)
- moved C22 127.9 mm to (151.5, 88.8), turned to -90 degrees
- moved SW6 119.3 mm to (91.1, 58.9)
- moved C28 116.9 mm to (151.5, 99.3), turned to -90 degrees
- moved C26 115.8 mm to (142.2, 80.5)
- moved C36 110.6 mm to (140.7, 65.6)
- moved C33 108.9 mm to (116.7, 128.0)
- moved SW5 104.2 mm to (99.1, 58.9)
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- renumbered J5 to J2, J6 to J3, J7 to J4, J2 to J5, J3 to J6, J8 to J7, J12 to J8, R12 to R10, R13 to R11, R14 to R12, R15 to R13, R16 to R14, R17 to R15, R8 to R6, R9 to R7, R10 to R8, R11 to R9, U13 to U12, U14 to U13, U9 to U2, U10 to U3, U11 to U4, U2 to U5, U3 to U6, U4 to U7, U12 to U8, U6 to U9
Connections:
- J11 pad 1: VDC -> /connectivity/ADCa_Pin
- J11 pad 2: GND -> ADCa
- J13 pad 1: ADCa -> /connectivity/ADCc_Pin
- J13 pad 2: ADCb -> ADCc
- J13 pad 3: ADCc -> Net-(J13-Pin_3)
- J14 pad 1: ADCa -> /connectivity/ADCd_Pin
- J14 pad 2: Net-(J14-Pin_2) -> ADCd
- J15 pad 1: ADCb -> /connectivity/ADCa_Pin
- J15 pad 2: Net-(J15-Pin_2) -> /connectivity/ADCb_Pin
- J17 pad 1: ADCd -> VDC
- J17 pad 2: Net-(J17-Pin_2) -> GND
- R10 pad 1: LEDa -> LEDc
- R11 pad 1: LEDa -> LEDd
- R9 pad 1: LEDa -> LEDb
- RV1 pad 2: Net-(J14-Pin_2) -> Net-(J11-Pin_3)
- RV2 pad 2: Net-(J15-Pin_2) -> Net-(J12-Pin_3)
- RV3 pad 2: Net-(J16-Pin_2) -> Net-(J13-Pin_3)
- RV4 pad 2: Net-(J17-Pin_2) -> Net-(J14-Pin_3)
Routing:
- net GND: track 0.00 -> 416.1 mm, vias 0 -> 50
- net +3.3V: track 0.00 -> 231.6 mm, vias 0 -> 42
- net ADCa: track 0.00 -> 159.8 mm, vias 0 -> 1
- net ADCb: track 0.00 -> 134.8 mm, vias 0 -> 1
- net ADCc: track 0.00 -> 107.9 mm, vias 0 -> 1
- net ADCd: track 0.00 -> 104.9 mm, vias 0 -> 1
- net VBUS: track 0.00 -> 104.3 mm, vias 0 -> 2
- net +5V: track 0.00 -> 87.6 mm, vias 0 -> 3
- net Net-(U1-BOOT0): track 0.00 -> 87.5 mm, vias 0 -> 4
- net USB_D-: track 0.00 -> 85.2 mm
- net USB_D+: track 0.00 -> 85.2 mm
- net Net-(U1-NRST): track 0.00 -> 77.2 mm, vias 0 -> 2
- net TIMd: track 0.00 -> 71.4 mm, vias 0 -> 1
- net LEDd: track 0.00 -> 71.4 mm, vias 0 -> 4
- net SWa: track 0.00 -> 69.4 mm, vias 0 -> 2
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- added copper zone on F.Cu, net +1V2
- added copper zone on F.Cu, net +3.3V
- added copper zone on In1.Cu, net +3.3V
- added copper zone on F.Cu, net GND
- added copper zone on In2.Cu, net GND
Other:
- board outline added: 151 x 90 mm
- copper layers 2 -> 4
- board text added: "Power Protection Circuits"
