File: dsp1_stm32/mcu_main.kicad_sch (KiCad schematic)
At the start: 11 parts, among them SW1 SW_Push, SW2 SW_SPDT, U1 STM32H757IITx, Y1 25MHz

Commit message: Circuit done
Other:
- note removed: "OPAMP1_VOUT internally connected to PC5 : ADC1_INN4_INP8"
- moved on the sheet: C1, C2, C3, C4, C5, R1, R2, SW1, SW2, U1, Y1

Commit message: Finished schematic
Parts:
- added D1: GREEN, LED_SMD:LED_0805_2012Metric, symbol Device:LED
- added R3: 470, Resistor_SMD:R_0603_1608Metric, symbol Device:R_US
- C1, C2: footprint (none) -> Capacitor_SMD:C_0402_1005Metric
- C3, C4, C5: footprint (none) -> Capacitor_SMD:C_0603_1608Metric
- R1, R2: footprint (none) -> Resistor_SMD:R_0603_1608Metric
- SW1: footprint (none) -> Button_Switch_SMD:SW_Push_1P1T_NO_CK_KMR2
- SW2: footprint (none) -> Button_Switch_SMD:Nidec_Copal_CAS-120A
- Y1: footprint (none) -> Crystal:Crystal_SMD_SeikoEpson_FA238-4Pin_3.2x2.5mm
Connections:
- net GND: now also D1.1 (K)
- net at R2.1, SW2.2 (B): now also R3.1
- net LEDa: now reaches U1.156 (PG12)
- net LEDb: now reaches U1.157 (PG13)
- net LEDc: now reaches U1.158 (PG14)
- net LEDd: now reaches U1.161 (PG15)
- new net: D1.2 (A), R3.2
- no-connect marks 78 -> 74
Other:
- moved on the sheet: R2

Commit message: PCB dsp v1 done
Parts:
- SW1: footprint Button_Switch_SMD:SW_Push_1P1T_NO_CK_KMR2 -> Button_Switch_SMD:SW_SPST_PTS647_Sx38
- SW2: footprint Button_Switch_SMD:Nidec_Copal_CAS-120A -> Button_Switch_SMD:SW_SPDT_PCM12
Changed lines of the file:
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@@
 			)
 		)
-		(property "Footprint" "Button_Switch_SMD:Nidec_Copal_CAS-120A"
+		(property "Footprint" "Button_Switch_SMD:SW_SPDT_PCM12"
 			(at 46.99 166.37 0)
 			(effects
@@
 			)
 		)
-		(property "Footprint" "Button_Switch_SMD:SW_Push_1P1T_NO_CK_KMR2"
+		(property "Footprint" "Button_Switch_SMD:SW_SPST_PTS647_Sx38"
 			(at 39.37 135.89 0)
 			(effects
