File: dsp1_stm32/power.kicad_sch (KiCad schematic)
At the start: 41 parts, among them U10 TLV62568DBV, U9 TLV62568DBV

Commit message: Circuit done
Connections:
- net +3.3V: no longer C15.1, C18.1, C21.1, C24.1
- net +3.3VA: now also C15.1, C18.1, C21.1, C24.1
Other:
- moved on the sheet: C10, C11, C12, C13, C14, C15, C16, C17, C18, C19, C20, C21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

Commit message: Finished schematic
Parts:
- removed JP5: Jumper_3_Bridged12, symbol Jumper:Jumper_3_Bridged12
- added J18: Conn_01x03_Pin, Connector_PinHeader_2.54mm:PinHeader_1x03_P2.54mm_Vertical, symbol Connector:Conn_01x03_Pin
- C10, C11, C19, C30, C36, C6, C7, C8, C9: footprint (none) -> Capacitor_SMD:C_0603_1608Metric
- C12: renamed from C15; footprint (none) -> Capacitor_SMD:C_0603_1608Metric
- C13: renamed from C12; footprint (none) -> Capacitor_SMD:C_0603_1608Metric
- C14: renamed from C18; footprint (none) -> Capacitor_SMD:C_0603_1608Metric
- C15: renamed from C21; footprint (none) -> Capacitor_SMD:C_0603_1608Metric
- C16: renamed from C13; footprint (none) -> Capacitor_SMD:C_0603_1608Metric
- C17: renamed from C24; footprint (none) -> Capacitor_SMD:C_0603_1608Metric
- C18: renamed from C16; footprint (none) -> Capacitor_SMD:C_0603_1608Metric
- C20: renamed from C22; footprint (none) -> Capacitor_SMD:C_0603_1608Metric
- C21: renamed from C26; footprint (none) -> Capacitor_SMD:C_0603_1608Metric
- C22: renamed from C14; footprint (none) -> Capacitor_SMD:C_0603_1608Metric
- C23: renamed from C25; footprint (none) -> Capacitor_SMD:C_0603_1608Metric
- C24: renamed from C28; footprint (none) -> Capacitor_SMD:C_0603_1608Metric
- C25: renamed from C17; footprint (none) -> Capacitor_SMD:C_0603_1608Metric
- C26: renamed from C27; footprint (none) -> Capacitor_SMD:C_0603_1608Metric
- C27: renamed from C29; footprint (none) -> Capacitor_SMD:C_0603_1608Metric
- C28: renamed from C31; footprint (none) -> Capacitor_SMD:C_0603_1608Metric
- C29: renamed from C20; footprint (none) -> Capacitor_SMD:C_0603_1608Metric
- C31: renamed from C33; footprint (none) -> Capacitor_SMD:C_0603_1608Metric
- C32: renamed from C23; footprint (none) -> Capacitor_SMD:C_0603_1608Metric
- C33: renamed from C32; footprint (none) -> Capacitor_SMD:C_0603_1608Metric
- C34: renamed from C35; footprint (none) -> Capacitor_SMD:C_0603_1608Metric
- C35: renamed from C34; footprint (none) -> Capacitor_SMD:C_0603_1608Metric
- FB1: footprint (none) -> Inductor_SMD:L_0603_1608Metric
- L1, L2: footprint (none) -> Inductor_SMD:L_0805_2012Metric
- R14: renamed from R9; footprint (none) -> Resistor_SMD:R_0603_1608Metric
- R15: renamed from R10; footprint (none) -> Resistor_SMD:R_0603_1608Metric
- R16: renamed from R11; footprint (none) -> Resistor_SMD:R_0603_1608Metric
- R17: renamed from R12; footprint (none) -> Resistor_SMD:R_0603_1608Metric
Connections:
- net +5V: now also J18.2 (Pin_2)
- net VBUS: now also J18.3 (Pin_3)
- net VDC: now also J18.1 (Pin_1)

Commit message: PCB dsp v1 done
Parts:
- added J16: USB_C_Receptacle_USB2.0_14P, Connector_USB:USB_C_Receptacle_GCT_USB4105-xx-A_16P_TopMnt_Horizontal, symbol Connector:USB_C_Receptacle_USB2.0_14P
- added J17: Jack-DC, Connector_BarrelJack:BarrelJack_Horizontal, symbol Connector:Jack-DC
- added R16, R17: 5.1k, Resistor_SMD:R_0603_1608Metric, symbol Device:R_US
- added U14: USBLC6-2SC6, Package_TO_SOT_SMD:SOT-23-6, symbol Power_Protection:USBLC6-2SC6
- renumbered R14 to R12, R15 to R13, R16 to R14, R17 to R15, U9 to U12, U10 to U13
Connections:
- net GND: now also J16.A1 (GND), J16.A12 (GND), J16.B1 (GND), J16.B12 (GND), J16.S1 (SHIELD), J17.2, R16.1, R17.1, U14.2 (GND)
- net VBUS: now also J16.A4 (VBUS), J16.A9 (VBUS), J16.B4 (VBUS), J16.B9 (VBUS), U14.5 (VBUS)
- net VDC: now also J17.1
- new net: J16.A5 (CC1), R16.2
- new net: J16.B5 (CC2), R17.2
- new net: J16.A6 (D+), J16.B6 (D+), U14.3 (I/O2)
- new net: J16.A7 (D-), J16.B7 (D-), U14.1 (I/O1)
- new net USB_D+: U14.4 (I/O2)
- new net USB_D-: U14.6 (I/O1)
Other:
- note added: "Add protection circuits here"
- moved on the sheet: C10, C11, C12, C13, C14, C15, C16, C17, C18, C19, C20, C21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
